Commit message: New updates: See wiki

File: nist_gear/robots/kitting/urdf/linear_arm_actuator.urdf.xacro (robot description, xacro)
@@ -2,5 +2,5 @@
 <robot xmlns:xacro="http://www.ros.org/wiki/xacro">
 <xacro:property name="base_len" value="0.2" />
-<xacro:property name="actuator_len" value="14" />
+<xacro:property name="actuator_len" value="10" />
 <xacro:property name="actuator_height" value="0.1" />
 <xacro:arg name="use_velocity_interface" default="false" />

Commit message: Features implemented and documentation added (see updates on wiki)

File: nist_gear/robots/kitting/urdf/linear_arm_actuator.urdf.xacro (robot description, xacro)
@@ -2,5 +2,5 @@
 <robot xmlns:xacro="http://www.ros.org/wiki/xacro">
 <xacro:property name="base_len" value="0.2" />
-<xacro:property name="actuator_len" value="14" />
+<xacro:property name="actuator_len" value="10" />
 <xacro:property name="actuator_height" value="0.1" />
 <xacro:arg name="use_velocity_interface" default="false" />
@@ -17,5 +17,5 @@
   </link>
   <gazebo reference="linear_arm_actuator">
-    <material>Gazebo/Grey</material>
+    <material>Gazebo/GreyTransparent</material>
   </gazebo>
   <joint name="linear_arm_actuator_joint" type="prismatic">
