Commit message: initial changes to work with ros iron

File: ariac_description/urdf/ceiling_robot/ceiling_robot_macro.xacro (robot description, xacro)
@@ -20,5 +20,5 @@
       rail_thickness="0.1"
       torso_height="-2.3"
-      initial_positions="${load_yaml(initial_positions_file)}"
+      initial_positions="${xacro.load_yaml(initial_positions_file)}"
       >
     </xacro:gantry>
@@ -26,5 +26,5 @@
     <xacro:ur_robot
       name="ceiling_arm"
-      prefix="ceiling_"
+      tf_prefix="ceiling_"
       parent="torso_main"
       joint_limits_parameters_file="$(find ur_description)/config/ur10e/joint_limits.yaml"
@@ -33,5 +33,5 @@
       visual_parameters_file="$(find ur_description)/config/ur10e/visual_parameters.yaml"
       sim_gazebo="true"
-      initial_positions="${load_yaml(initial_positions_file)}">
+      initial_positions="${xacro.load_yaml(initial_positions_file)}">
       <origin xyz="0.51 0.0 1.3" rpy="0 1.57 0" />
     </xacro:ur_robot>

File: ariac_description/urdf/floor_robot/floor_robot_macro.xacro (robot description, xacro)
@@ -13,5 +13,5 @@
     <xacro:linear_actuator
       parent="world"
-      initial_positions="${load_yaml(initial_positions_file)}"
+      initial_positions="${xacro.load_yaml(initial_positions_file)}"
       >
     </xacro:linear_actuator>
@@ -19,5 +19,5 @@
     <xacro:ur_robot
       name="floor_arm"
-      prefix="floor_"
+      tf_prefix="floor_"
       parent="robot_base"
       joint_limits_parameters_file="$(find ur_description)/config/ur10e/joint_limits.yaml"
@@ -26,5 +26,5 @@
       visual_parameters_file="$(find ur_description)/config/ur10e/visual_parameters.yaml"
       sim_gazebo="true"
-      initial_positions="${load_yaml(initial_positions_file)}">
+      initial_positions="${xacro.load_yaml(initial_positions_file)}">
       <origin xyz="0 0 0.05" rpy="0 0 0" />
     </xacro:ur_robot>

File: ariac_description/urdf/floor_robot/linear_actuator_macro.xacro (robot description, xacro)
@@ -47,5 +47,5 @@
       <parent link="slide_bar"/>
       <child link="robot_base"/>
-      <limit effort="1000.0" lower="-4.8" upper="4.8" velocity="4"/>
+      <limit effort="1000.0" lower="-4.8" upper="4.8" velocity="4" acceleration="0.5"/>
       <dynamics damping="20.0" friction="500.0" />
     </joint>

Commit message: fix robot initial poses

File: ariac_description/urdf/ceiling_robot/ceiling_robot_macro.xacro (robot description, xacro)
@@ -7,6 +7,5 @@
     <!-- Inclue gripper macro -->
     <xacro:include filename="$(find ariac_description)/urdf/vacuum_gripper/vacuum_gripper_macro.xacro"/>
-    <xacro:arg name="initial_positions_file" default="$(find ariac_description)/config/ceiling_robot_initial_positions.yaml"/>
-    <xacro:property name="initial_positions_file" default="$(arg initial_positions_file)"/>
+    <xacro:property name="initial_positions_file" default="$(find ariac_description)/config/ceiling_robot_initial_positions.yaml"/>
     <!-- Run gantry macro -->
     <xacro:gantry

File: ariac_description/urdf/ceiling_robot/gantry.ros2_control.xacro (robot description, xacro)
@@ -3,5 +3,6 @@
   <xacro:macro name="gantry_ros2_control" params="
     name
-    initial_positions">
+    initial_positions:=${dict(gantry_x_axis_joint=0.0)}
+    ">
     <ros2_control name="${name}" type="system">
       <hardware>
@@ -18,5 +19,5 @@
         </command_interface>
         <state_interface name="position">
-          <param name="initial_value">0</param>
+          <param name="initial_value">${initial_positions['gantry_x_axis_joint']}</param>
         </state_interface>
         <state_interface name="velocity"/>
@@ -33,5 +34,5 @@
         </command_interface>
         <state_interface name="position">
-          <param name="initial_value">0</param>
+          <param name="initial_value">${initial_positions['gantry_y_axis_joint']}</param>
         </state_interface>
         <state_interface name="velocity"/>
@@ -48,5 +49,5 @@
         </command_interface>
         <state_interface name="position">
-          <param name="initial_value">0</param>
+          <param name="initial_value">${initial_positions['gantry_rotation_joint']}</param>
         </state_interface>
         <state_interface name="velocity"/>

File: ariac_description/urdf/floor_robot/floor_robot_macro.xacro (robot description, xacro)
@@ -8,6 +8,5 @@
     <!-- Inclue gripper macro -->
     <xacro:include filename="$(find ariac_description)/urdf/vacuum_gripper/vacuum_gripper_macro.xacro"/>
-    <xacro:arg name="initial_positions_file" default="$(find ariac_description)/config/floor_robot_initial_positions.yaml"/>
-    <xacro:property name="initial_positions_file" default="$(arg initial_positions_file)"/>
+    <xacro:property name="initial_positions_file" default="$(find ariac_description)/config/floor_robot_initial_positions.yaml"/>
     <!-- Run linear actuator macro -->
     <xacro:linear_actuator

File: ariac_description/urdf/floor_robot/linear_actuator.ros2_control.xacro (robot description, xacro)
@@ -14,5 +14,5 @@
       </command_interface>
       <state_interface name="position">
-        <param name="initial_value">0</param>
+        <param name="initial_value">${initial_positions['linear_actuator']}</param>
       </state_interface>
       <state_interface name="velocity"/>
