Commit message: added camera mount to xacro

File: ariac_description/urdf/ariac_robots/ariac_robots.urdf.xacro (robot description, xacro)
@@ -6,4 +6,10 @@
   <material name="Grey">
     <color rgba="${220/255} ${220/255} ${220/255} 1.0"/>
+  </material>
+  <material name="Black">
+    <color rgba="${240/255} ${240/255} ${240/255} 1.0"/>
+  </material>
+  <material name="white">
+    <color rgba="${20/255} ${20/255} ${20/255} 1.0"/>
   </material>
   <!-- Locate Robot Macros -->

File: ariac_description/urdf/vacuum_gripper/vacuum_gripper_macro.xacro (robot description, xacro)
@@ -15,5 +15,4 @@
         <origin xyz="0 0 -0.005" rpy="0 0 0"/>
         <geometry>
-          <!-- <mesh filename="file://$(find ariac_description)/meshes/vacuum_gripper/vacuum_gripper.stl" scale="1 1 1"/> -->
           <cylinder radius="0.05" length="0.01" />
         </geometry>
@@ -25,4 +24,21 @@
       </inertial>
     </link>
+    <link name ="${prefix}_camera_link">
+      <visual>
+        <origin xyz="0 0 -.06" rpy="1.57 0 0"/>
+        <geometry>
+          <mesh filename="file://$(find ariac_description)/meshes/vacuum_gripper/camera_mount.stl" scale="1 1 1"/>
+        </geometry>
+      </visual>
+      <visual>
+        <origin xyz="0 .06 -.03" rpy="1.57 0 0"/>
+        <geometry>
+          <sphere radius=".01"/>
+        </geometry>
+      </visual>
+    </link>
+    <gazebo reference="${prefix}_camera_link">
+      <material>Gazebo/Orange</material>
+    </gazebo>
     <gazebo reference="${prefix}_gripper">
       <visual name="${prefix}_gripper_visual">
@@ -34,7 +50,4 @@
       </visual>
     </gazebo>
-    <gazebo reference="${prefix}_gripper">
-      <material>Gazebo/Black</material>
-    </gazebo>
     <joint name="${prefix}_gripper_joint" type="revolute">
       <axis xyz="0 0 1"/>
@@ -43,4 +56,10 @@
       <limit lower="-.001" upper=".001" effort="1000" velocity="0" />
       <origin xyz="0.0 0.0 0.01" rpy="0.0 0.0 0.0"/>
+    </joint>
+    <joint name="${prefix}_camera_joint" type="fixed">
+      <axis xyz="0 1 0" />
+      <origin xyz="0 0 0" rpy="0 0 0"/>
+      <parent link="${prefix}_gripper"/>
+      <child link="${prefix}_camera_link"/>
     </joint>
     <!-- Add a contact sensor to the gripper -->

Commit message: added camera sensors and proper xacro arguments

File: ariac_description/urdf/ariac_robots/ariac_robots.urdf.xacro (robot description, xacro)
@@ -17,8 +17,23 @@
   <xacro:include filename="$(find ariac_description)/urdf/ceiling_robot/ceiling_robot_macro.xacro"/>
   <xacro:include filename="$(find ariac_description)/urdf/agv/agv_macro.xacro"/>
+  <!-- Define arguments for robot cameras -->
+  <xacro:arg name="floor_robot_camera_active_arg" default="false"/>
+  <xacro:property name="floor_robot_camera_active" value="$(arg floor_robot_camera_active_arg)" />
+  <xacro:arg name="floor_robot_camera_type_arg" default="rgb"/>
+  <xacro:property name="floor_robot_camera_type" value="$(arg floor_robot_camera_type_arg)" />
+  <xacro:arg name="ceiling_robot_camera_active_arg" default="false"/>
+  <xacro:property name="ceiling_robot_camera_active" value="$(arg ceiling_robot_camera_active_arg)" />
+  <xacro:arg name="ceiling_robot_camera_type_arg" default="rgb"/>
+  <xacro:property name="ceiling_robot_camera_type" value="$(arg ceiling_robot_camera_type_arg)" />
   <!-- Floor Robot -->
-  <xacro:floor_robot/>
+  <xacro:floor_robot
+    camera_active="${floor_robot_camera_active}"
+    camera_type="${floor_robot_camera_type}">
+  </xacro:floor_robot>
   <!-- Ceiling Robot -->
-  <xacro:ceiling_robot/>
+  <xacro:ceiling_robot
+    camera_active="${ceiling_robot_camera_active}"
+    camera_type="${ceiling_robot_camera_type}">
+  </xacro:ceiling_robot>
   <!-- AGV1 -->
   <xacro:agv

File: ariac_description/urdf/ceiling_robot/ceiling_robot_macro.xacro (robot description, xacro)
@@ -1,5 +1,8 @@
 <?xml version="1.0" ?>
 <robot xmlns:xacro="http://wiki.ros.org/xacro">
-  <xacro:macro name="ceiling_robot" params="">
+  <xacro:macro name="ceiling_robot" params="
+    camera_active
+    camera_type
+  ">
     <xacro:include filename="$(find ariac_description)/urdf/ceiling_robot/gantry_macro.xacro"/>
     <!-- Inclue ur robot macro -->
@@ -7,6 +10,5 @@
     <!-- Inclue gripper macro -->
     <xacro:include filename="$(find ariac_description)/urdf/vacuum_gripper/vacuum_gripper_macro.xacro"/>
-    <xacro:arg name="initial_positions_file" default="$(find ariac_description)/config/ceiling_robot_initial_positions.yaml"/>
-    <xacro:property name="initial_positions_file" default="$(arg initial_positions_file)"/>
+    <xacro:property name="initial_positions_file" default="$(find ariac_description)/config/ceiling_robot_initial_positions.yaml"/>
     <!-- Run gantry macro -->
     <xacro:gantry
@@ -40,4 +42,6 @@
       parent="wrist_3_link"
       prefix="ceiling"
+      use_camera="${camera_active}"
+      camera_type="${camera_type}"
       >
     </xacro:vacuum_gripper>

File: ariac_description/urdf/floor_robot/floor_robot_macro.xacro (robot description, xacro)
@@ -1,5 +1,8 @@
 <?xml version="1.0" ?>
 <robot xmlns:xacro="http://wiki.ros.org/xacro">
-  <xacro:macro name="floor_robot" params="">
+  <xacro:macro name="floor_robot" params="
+    camera_active
+    camera_type
+  ">
     <!-- Include linear actuator macro -->
     <xacro:include filename="$(find ariac_description)/urdf/floor_robot/linear_actuator_macro.xacro"/>
@@ -8,6 +11,5 @@
     <!-- Inclue gripper macro -->
     <xacro:include filename="$(find ariac_description)/urdf/vacuum_gripper/vacuum_gripper_macro.xacro"/>
-    <xacro:arg name="initial_positions_file" default="$(find ariac_description)/config/floor_robot_initial_positions.yaml"/>
-    <xacro:property name="initial_positions_file" default="$(arg initial_positions_file)"/>
+    <xacro:property name="initial_positions_file" default="$(find ariac_description)/config/floor_robot_initial_positions.yaml"/>
     <!-- Run linear actuator macro -->
     <xacro:linear_actuator
@@ -33,4 +35,6 @@
       parent="wrist_3_link"
       prefix="floor"
+      use_camera="${camera_active}"
+      camera_type="${camera_type}"
       >
     </xacro:vacuum_gripper>

File: ariac_description/urdf/vacuum_gripper/vacuum_gripper_macro.xacro (robot description, xacro)
@@ -4,5 +4,6 @@
     parent
     prefix
-    use_camera:=true
+    use_camera
+    camera_type
     ">
     <!-- Gripper Link -->
@@ -76,5 +77,6 @@
     <!-- Camera -->
     <xacro:if value="${use_camera}">
-      <link name ="${prefix}_camera_mount_link">
+      <!-- Mount Link -->
+      <link name ="${prefix}_robot_camera_mount_link">
         <visual>
           <origin xyz="0 0 0" rpy="0 0 0"/>
@@ -84,7 +86,8 @@
         </visual>
       </link>
-      <link name ="${prefix}_camera_link">
+      <!-- Camera Link -->
+      <link name ="${prefix}_robot_camera_link">
         <visual>
-          <origin xyz="0 0 0" rpy="0 0 0"/>
+          <origin xyz="0 0 0" rpy="1.57 0 1.57"/>
           <geometry>
             <mesh filename="file://$(find ariac_description)/meshes/vacuum_gripper/camera.stl" scale="1 1 1"/>
@@ -93,22 +96,87 @@
       </link>
       <!-- Add camera mount joint -->
-      <joint name="${prefix}_camera_mount_joint" type="fixed">
+      <joint name="${prefix}_robot_camera_mount_joint" type="fixed">
         <axis xyz="0 1 0" />
-        <origin xyz="0 0 -0.012" rpy="0 0 3.14"/>
+        <origin xyz="0 0 -0.012" rpy="0 0 0"/>
         <parent link="${prefix}_gripper"/>
-        <child link="${prefix}_camera_mount_link"/>
+        <child link="${prefix}_robot_camera_mount_link"/>
       </joint>
-      <joint name="${prefix}_camera_joint" type="fixed">
+      <!-- Add camera joint -->
+      <joint name="${prefix}_robot_camera_joint" type="fixed">
         <axis xyz="0 1 0" />
-        <origin xyz="0 -.07 -.006" rpy="0 0 0"/>
-        <parent link="${prefix}_camera_mount_link"/>
-        <child link="${prefix}_camera_link"/>
+        <origin xyz="0 -.07 -.006" rpy="0 -1.57 1.57"/>
+        <parent link="${prefix}_robot_camera_mount_link"/>
+        <child link="${prefix}_robot_camera_link"/>
       </joint>
       <!-- Add color to links -->
-      <gazebo reference="${prefix}_camera_mount_link">
+      <gazebo reference="${prefix}_robot_camera_mount_link">
         <material>Gazebo/Black</material>
       </gazebo>
-      <gazebo reference="${prefix}_camera_link">
+      <gazebo reference="${prefix}_robot_camera_link">
         <material>Gazebo/White</material>
+      </gazebo>
+      <!-- Add gazebo sensors -->
+      <xacro:property name="type" value="${camera_type}"/>
+      <gazebo reference="${prefix}_robot_camera_link">
+        <!-- Add rgb camera -->
+        <xacro:if value="${type == 'rgb'}">
+          <sensor type="camera" name="rgb_camera">
+            <always_on>true</always_on>
+            <visualize>false</visualize>
+            <update_rate>30</update_rate>
+            <camera name="${prefix}_robot_camera">
+              <horizontal_fov>1.5</horizontal_fov>
+              <image>
+                <width>640</width>
+                <height>480</height>
+                <format>R8G8B8</format>
+              </image>
+              <clip>
+                <near>0.1</near>
+                <far>10</far>
+              </clip>
+            </camera>
+            <plugin name="${prefix}_robot_camera_plugin" filename="libAriacCameraPlugin.so">
+              <ros>
+                <namespace></namespace>
+              </ros>
+              <camera_type>rgb</camera_type>
+              <camera_name>${prefix}_robot_camera</camera_name>
+              <frame_name>${prefix}_robot_camera_link</frame_name>
+            </plugin>
+          </sensor>
+        </xacro:if>
+        <xacro:if value="${type == 'rgbd'}">
+          <sensor type="depth" name="rgbd_camera">
+            <always_on>true</always_on>
+            <visualize>false</visualize>
+            <update_rate>30</update_rate>
+            <camera name="${prefix}_robot_camera">
+              <horizontal_fov>1.5</horizontal_fov>
+              <image>
+                <width>640</width>
+                <height>480</height>
+                <format>R8G8B8</format>
+              </image>
+              <clip>
+                <near>0.1</near>
+                <far>10</far>
+              </clip>
+              <noise>
+                <type>gaussian</type>
+                <mean>0.0</mean>
+                <stddev>0.001</stddev>
+              </noise>
+            </camera>
+            <plugin name="${prefix}_robot_camera_plugin" filename="libAriacCameraPlugin.so">
+              <ros>
+                <namespace></namespace>
+              </ros>
+              <camera_type>rgbd</camera_type>
+              <camera_name>${prefix}_robot_camera</camera_name>
+              <frame_name>${prefix}_robot_camera_link</frame_name>
+            </plugin>
+          </sensor>
+        </xacro:if>
       </gazebo>
     </xacro:if>

Commit message: Robot End-Effector Cameras (#274)
* Fix conveyor spawn part naming issue

* added camera mount to xacro

* improved visuals of camera and mount

* added camera sensors and proper xacro arguments

* update moveit_test launch file to match competitor.launch

File: ariac_description/urdf/ariac_robots/ariac_robots.urdf.xacro (robot description, xacro)
@@ -7,12 +7,33 @@
     <color rgba="${220/255} ${220/255} ${220/255} 1.0"/>
   </material>
+  <material name="Black">
+    <color rgba="${240/255} ${240/255} ${240/255} 1.0"/>
+  </material>
+  <material name="white">
+    <color rgba="${20/255} ${20/255} ${20/255} 1.0"/>
+  </material>
   <!-- Locate Robot Macros -->
   <xacro:include filename="$(find ariac_description)/urdf/floor_robot/floor_robot_macro.xacro"/>
   <xacro:include filename="$(find ariac_description)/urdf/ceiling_robot/ceiling_robot_macro.xacro"/>
   <xacro:include filename="$(find ariac_description)/urdf/agv/agv_macro.xacro"/>
+  <!-- Define arguments for robot cameras -->
+  <xacro:arg name="floor_robot_camera_active_arg" default="false"/>
+  <xacro:property name="floor_robot_camera_active" value="$(arg floor_robot_camera_active_arg)" />
+  <xacro:arg name="floor_robot_camera_type_arg" default="rgb"/>
+  <xacro:property name="floor_robot_camera_type" value="$(arg floor_robot_camera_type_arg)" />
+  <xacro:arg name="ceiling_robot_camera_active_arg" default="false"/>
+  <xacro:property name="ceiling_robot_camera_active" value="$(arg ceiling_robot_camera_active_arg)" />
+  <xacro:arg name="ceiling_robot_camera_type_arg" default="rgb"/>
+  <xacro:property name="ceiling_robot_camera_type" value="$(arg ceiling_robot_camera_type_arg)" />
   <!-- Floor Robot -->
-  <xacro:floor_robot/>
+  <xacro:floor_robot
+    camera_active="${floor_robot_camera_active}"
+    camera_type="${floor_robot_camera_type}">
+  </xacro:floor_robot>
   <!-- Ceiling Robot -->
-  <xacro:ceiling_robot/>
+  <xacro:ceiling_robot
+    camera_active="${ceiling_robot_camera_active}"
+    camera_type="${ceiling_robot_camera_type}">
+  </xacro:ceiling_robot>
   <!-- AGV1 -->
   <xacro:agv

File: ariac_description/urdf/ceiling_robot/ceiling_robot_macro.xacro (robot description, xacro)
@@ -1,5 +1,8 @@
 <?xml version="1.0" ?>
 <robot xmlns:xacro="http://wiki.ros.org/xacro">
-  <xacro:macro name="ceiling_robot" params="">
+  <xacro:macro name="ceiling_robot" params="
+    camera_active
+    camera_type
+  ">
     <xacro:include filename="$(find ariac_description)/urdf/ceiling_robot/gantry_macro.xacro"/>
     <!-- Inclue ur robot macro -->
@@ -39,4 +42,6 @@
       parent="wrist_3_link"
       prefix="ceiling"
+      use_camera="${camera_active}"
+      camera_type="${camera_type}"
       >
     </xacro:vacuum_gripper>

File: ariac_description/urdf/floor_robot/floor_robot_macro.xacro (robot description, xacro)
@@ -1,5 +1,8 @@
 <?xml version="1.0" ?>
 <robot xmlns:xacro="http://wiki.ros.org/xacro">
-  <xacro:macro name="floor_robot" params="">
+  <xacro:macro name="floor_robot" params="
+    camera_active
+    camera_type
+  ">
     <!-- Include linear actuator macro -->
     <xacro:include filename="$(find ariac_description)/urdf/floor_robot/linear_actuator_macro.xacro"/>
@@ -32,4 +35,6 @@
       parent="wrist_3_link"
       prefix="floor"
+      use_camera="${camera_active}"
+      camera_type="${camera_type}"
       >
     </xacro:vacuum_gripper>

File: ariac_description/urdf/vacuum_gripper/vacuum_gripper_macro.xacro (robot description, xacro)
@@ -3,5 +3,9 @@
   <xacro:macro name="vacuum_gripper" params="
     parent
-    prefix">
+    prefix
+    use_camera
+    camera_type
+    ">
+    <!-- Gripper Link -->
     <link name="${prefix}_gripper">
       <visual name="${prefix}_gripper_visual">
@@ -15,26 +19,14 @@
         <origin xyz="0 0 -0.005" rpy="0 0 0"/>
         <geometry>
-          <!-- <mesh filename="file://$(find ariac_description)/meshes/vacuum_gripper/vacuum_gripper.stl" scale="1 1 1"/> -->
           <cylinder radius="0.05" length="0.01" />
         </geometry>
       </collision>
       <inertial>
-        <origin xyz="0 0 0" rpy="0 0 0"/>
-        <mass value="0.01"/>
-        <inertia ixx="0.0000063" ixy="0.0" ixz="0.0" iyy="0.0000063" iyz="0.0" izz="0.000025"/>
+        <origin xyz="0 0 -0.005" rpy="0 0 0"/>
+        <mass value="0.102"/>
+        <inertia ixx="0.0000647" ixy="0.0" ixz="0.0" iyy="0.0000647" iyz="0.0" izz="0.0001276"/>
       </inertial>
     </link>
-    <gazebo reference="${prefix}_gripper">
-      <visual name="${prefix}_gripper_visual">
-        <plugin filename="libGripperColorPlugin.so" name="${prefix}_gripper_color_plugin">
-          <ros>
-          </ros>
-          <robot_name>${prefix}_robot</robot_name>
-        </plugin>
-      </visual>
-    </gazebo>
-    <gazebo reference="${prefix}_gripper">
-      <material>Gazebo/Black</material>
-    </gazebo>
+    <!-- Gripper Joint -->
     <joint name="${prefix}_gripper_joint" type="revolute">
       <axis xyz="0 0 1"/>
@@ -53,4 +45,5 @@
       </sensor>
     </gazebo>
+    <!-- Vacuum gripper plugin -->
     <gazebo>
       <plugin filename="libVacuumGripperPlugin.so" name="${prefix}_vacuum_gripper_plugin">
@@ -61,4 +54,15 @@
       </plugin>
     </gazebo>
+    <!-- Color change plugin -->
+    <gazebo reference="${prefix}_gripper">
+      <visual name="${prefix}_gripper_visual">
+        <plugin filename="libGripperColorPlugin.so" name="${prefix}_gripper_color_plugin">
+          <ros>
+          </ros>
+          <robot_name>${prefix}_robot</robot_name>
+        </plugin>
+      </visual>
+    </gazebo>
+    <!-- ROS2 Control for the gripper joint -->
     <ros2_control name="${prefix}_gripper_control" type="system">
       <hardware>
@@ -71,4 +75,110 @@
       </joint>
     </ros2_control>
+    <!-- Camera -->
+    <xacro:if value="${use_camera}">
+      <!-- Mount Link -->
+      <link name ="${prefix}_robot_camera_mount_link">
+        <visual>
+          <origin xyz="0 0 0" rpy="0 0 0"/>
+          <geometry>
+            <mesh filename="file://$(find ariac_description)/meshes/vacuum_gripper/camera_mount.stl" scale="1 1 1"/>
+          </geometry>
+        </visual>
+      </link>
+      <!-- Camera Link -->
+      <link name ="${prefix}_robot_camera_link">
+        <visual>
+          <origin xyz="0 0 0" rpy="1.57 0 1.57"/>
+          <geometry>
+            <mesh filename="file://$(find ariac_description)/meshes/vacuum_gripper/camera.stl" scale="1 1 1"/>
+          </geometry>
+        </visual>
+      </link>
+      <!-- Add camera mount joint -->
+      <joint name="${prefix}_robot_camera_mount_joint" type="fixed">
+        <axis xyz="0 1 0" />
+        <origin xyz="0 0 -0.012" rpy="0 0 0"/>
+        <parent link="${prefix}_gripper"/>
+        <child link="${prefix}_robot_camera_mount_link"/>
+      </joint>
+      <!-- Add camera joint -->
+      <joint name="${prefix}_robot_camera_joint" type="fixed">
+        <axis xyz="0 1 0" />
+        <origin xyz="0 -.07 -.006" rpy="0 -1.57 1.57"/>
+        <parent link="${prefix}_robot_camera_mount_link"/>
+        <child link="${prefix}_robot_camera_link"/>
+      </joint>
+      <!-- Add color to links -->
+      <gazebo reference="${prefix}_robot_camera_mount_link">
+        <material>Gazebo/Black</material>
+      </gazebo>
+      <gazebo reference="${prefix}_robot_camera_link">
+        <material>Gazebo/White</material>
+      </gazebo>
+      <!-- Add gazebo sensors -->
+      <xacro:property name="type" value="${camera_type}"/>
+      <gazebo reference="${prefix}_robot_camera_link">
+        <!-- Add rgb camera -->
+        <xacro:if value="${type == 'rgb'}">
+          <sensor type="camera" name="rgb_camera">
+            <always_on>true</always_on>
+            <visualize>false</visualize>
+            <update_rate>30</update_rate>
+            <camera name="${prefix}_robot_camera">
+              <horizontal_fov>1.5</horizontal_fov>
+              <image>
+                <width>640</width>
+                <height>480</height>
+                <format>R8G8B8</format>
+              </image>
+              <clip>
+                <near>0.1</near>
+                <far>10</far>
+              </clip>
+            </camera>
+            <plugin name="${prefix}_robot_camera_plugin" filename="libAriacCameraPlugin.so">
+              <ros>
+                <namespace></namespace>
+              </ros>
+              <camera_type>rgb</camera_type>
+              <camera_name>${prefix}_robot_camera</camera_name>
+              <frame_name>${prefix}_robot_camera_link</frame_name>
+            </plugin>
+          </sensor>
+        </xacro:if>
+        <xacro:if value="${type == 'rgbd'}">
+          <sensor type="depth" name="rgbd_camera">
+            <always_on>true</always_on>
+            <visualize>false</visualize>
+            <update_rate>30</update_rate>
+            <camera name="${prefix}_robot_camera">
+              <horizontal_fov>1.5</horizontal_fov>
+              <image>
+                <width>640</width>
+                <height>480</height>
+                <format>R8G8B8</format>
+              </image>
+              <clip>
+                <near>0.1</near>
+                <far>10</far>
+              </clip>
+              <noise>
+                <type>gaussian</type>
+                <mean>0.0</mean>
+                <stddev>0.001</stddev>
+              </noise>
+            </camera>
+            <plugin name="${prefix}_robot_camera_plugin" filename="libAriacCameraPlugin.so">
+              <ros>
+                <namespace></namespace>
+              </ros>
+              <camera_type>rgbd</camera_type>
+              <camera_name>${prefix}_robot_camera</camera_name>
+              <frame_name>${prefix}_robot_camera_link</frame_name>
+            </plugin>
+          </sensor>
+        </xacro:if>
+      </gazebo>
+    </xacro:if>
   </xacro:macro>
 </robot>
