Commit message: improved visuals of camera and mount

File: ariac_description/urdf/vacuum_gripper/vacuum_gripper_macro.xacro (robot description, xacro)
@@ -3,5 +3,8 @@
   <xacro:macro name="vacuum_gripper" params="
     parent
-    prefix">
+    prefix
+    use_camera:=true
+    ">
+    <!-- Gripper Link -->
     <link name="${prefix}_gripper">
       <visual name="${prefix}_gripper_visual">
@@ -19,35 +22,10 @@
       </collision>
       <inertial>
-        <origin xyz="0 0 0" rpy="0 0 0"/>
-        <mass value="0.01"/>
-        <inertia ixx="0.0000063" ixy="0.0" ixz="0.0" iyy="0.0000063" iyz="0.0" izz="0.000025"/>
+        <origin xyz="0 0 -0.005" rpy="0 0 0"/>
+        <mass value="0.102"/>
+        <inertia ixx="0.0000647" ixy="0.0" ixz="0.0" iyy="0.0000647" iyz="0.0" izz="0.0001276"/>
       </inertial>
     </link>
-    <link name ="${prefix}_camera_link">
-      <visual>
-        <origin xyz="0 0 -.06" rpy="1.57 0 0"/>
-        <geometry>
-          <mesh filename="file://$(find ariac_description)/meshes/vacuum_gripper/camera_mount.stl" scale="1 1 1"/>
-        </geometry>
-      </visual>
-      <visual>
-        <origin xyz="0 .06 -.03" rpy="1.57 0 0"/>
-        <geometry>
-          <sphere radius=".01"/>
-        </geometry>
-      </visual>
-    </link>
-    <gazebo reference="${prefix}_camera_link">
-      <material>Gazebo/Orange</material>
-    </gazebo>
-    <gazebo reference="${prefix}_gripper">
-      <visual name="${prefix}_gripper_visual">
-        <plugin filename="libGripperColorPlugin.so" name="${prefix}_gripper_color_plugin">
-          <ros>
-          </ros>
-          <robot_name>${prefix}_robot</robot_name>
-        </plugin>
-      </visual>
-    </gazebo>
+    <!-- Gripper Joint -->
     <joint name="${prefix}_gripper_joint" type="revolute">
       <axis xyz="0 0 1"/>
@@ -56,10 +34,4 @@
       <limit lower="-.001" upper=".001" effort="1000" velocity="0" />
       <origin xyz="0.0 0.0 0.01" rpy="0.0 0.0 0.0"/>
-    </joint>
-    <joint name="${prefix}_camera_joint" type="fixed">
-      <axis xyz="0 1 0" />
-      <origin xyz="0 0 0" rpy="0 0 0"/>
-      <parent link="${prefix}_gripper"/>
-      <child link="${prefix}_camera_link"/>
     </joint>
     <!-- Add a contact sensor to the gripper -->
@@ -72,4 +44,5 @@
       </sensor>
     </gazebo>
+    <!-- Vacuum gripper plugin -->
     <gazebo>
       <plugin filename="libVacuumGripperPlugin.so" name="${prefix}_vacuum_gripper_plugin">
@@ -80,4 +53,15 @@
       </plugin>
     </gazebo>
+    <!-- Color change plugin -->
+    <gazebo reference="${prefix}_gripper">
+      <visual name="${prefix}_gripper_visual">
+        <plugin filename="libGripperColorPlugin.so" name="${prefix}_gripper_color_plugin">
+          <ros>
+          </ros>
+          <robot_name>${prefix}_robot</robot_name>
+        </plugin>
+      </visual>
+    </gazebo>
+    <!-- ROS2 Control for the gripper joint -->
     <ros2_control name="${prefix}_gripper_control" type="system">
       <hardware>
@@ -90,4 +74,43 @@
       </joint>
     </ros2_control>
+    <!-- Camera -->
+    <xacro:if value="${use_camera}">
+      <link name ="${prefix}_camera_mount_link">
+        <visual>
+          <origin xyz="0 0 0" rpy="0 0 0"/>
+          <geometry>
+            <mesh filename="file://$(find ariac_description)/meshes/vacuum_gripper/camera_mount.stl" scale="1 1 1"/>
+          </geometry>
+        </visual>
+      </link>
+      <link name ="${prefix}_camera_link">
+        <visual>
+          <origin xyz="0 0 0" rpy="0 0 0"/>
+          <geometry>
+            <mesh filename="file://$(find ariac_description)/meshes/vacuum_gripper/camera.stl" scale="1 1 1"/>
+          </geometry>
+        </visual>
+      </link>
+      <!-- Add camera mount joint -->
+      <joint name="${prefix}_camera_mount_joint" type="fixed">
+        <axis xyz="0 1 0" />
+        <origin xyz="0 0 -0.012" rpy="0 0 3.14"/>
+        <parent link="${prefix}_gripper"/>
+        <child link="${prefix}_camera_mount_link"/>
+      </joint>
+      <joint name="${prefix}_camera_joint" type="fixed">
+        <axis xyz="0 1 0" />
+        <origin xyz="0 -.07 -.006" rpy="0 0 0"/>
+        <parent link="${prefix}_camera_mount_link"/>
+        <child link="${prefix}_camera_link"/>
+      </joint>
+      <!-- Add color to links -->
+      <gazebo reference="${prefix}_camera_mount_link">
+        <material>Gazebo/Black</material>
+      </gazebo>
+      <gazebo reference="${prefix}_camera_link">
+        <material>Gazebo/White</material>
+      </gazebo>
+    </xacro:if>
   </xacro:macro>
 </robot>

Commit message: switched gripper_joint to fixed and removed from moveit_config

File: ariac_description/urdf/vacuum_gripper/vacuum_gripper_macro.xacro (robot description, xacro)
@@ -29,11 +29,12 @@
     </link>
     <!-- Gripper Joint -->
-    <joint name="${prefix}_gripper_joint" type="revolute">
-      <axis xyz="0 0 1"/>
+    <joint name="${prefix}_gripper_joint" type="fixed">
       <parent link="${prefix}_${parent}"/>
       <child link="${prefix}_gripper"/>
-      <limit lower="-.001" upper=".001" effort="1000" velocity="0" />
       <origin xyz="0.0 0.0 0.01" rpy="0.0 0.0 0.0"/>
     </joint>
+    <gazebo reference='${prefix}_gripper_joint'>
+      <preserveFixedJoint>true</preserveFixedJoint>
+    </gazebo>
     <!-- Add a contact sensor to the gripper -->
     <gazebo reference="${prefix}_gripper">
